File: Board/Igniters.kicad_sch (KiCad schematic)
At the start: 54 parts, among them J2 Screw_Terminal_01x02, J3 Screw_Terminal_01x02, J4 Screw_Terminal_01x02, J5 Screw_Terminal_01x02, J6 Screw_Terminal_01x02, J7 Screw_Terminal_01x02, Q1 DO2300B, Q2 DO2300B, Q3 DO2300B, Q4 DO2300B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

Commit message: BOM update
Parts:
- D10, D11, D14, D15, D6, D7: MPN (none) -> GL0805UR01
- D12, D13, D4, D5, D8, D9: footprint Diode_SMD:D_0603_1608Metric -> Diode_SMD:D_MiniMELF; MPN (none) -> ZMM3V0-TD
- F1, F2, F3, F4, F5, F6: MPN (none) -> CF06V5TR50
- J2, J3, J4, J5, J6, J7: MPN (none) -> KF301-2P; now in the parts list
- Q1, Q2, Q3, Q4, Q5, Q6: MPN (none) -> DO2300B
- R31, R32, R39, R40, R47, R48: MPN (none) -> 1RC0603J0100; now in the parts list
- R33, R35, R41, R43, R49, R51: MPN (none) -> CL0603JN100KP; now in the parts list
- R34, R36, R37, R38, R42, R44, R45, R46, R50, R52, R53, R54: MPN (none) -> FRC0603F1002TS; now in the parts list
