File: Board/Interfaces.kicad_sch (KiCad schematic)
At the start: 32 parts, among them J10 Conn_Coaxial, J11 Conn_Coaxial, J12 USB_C_Receptacle_USB2.0_16P, J13 MEM2052-00-195-00-A_REVA, J8 Conn_01x02_Pin, J9 Conn_01x02_Pin, U16 E220-400M22S, U17 E220-400M22S, U18 74LVC2G04LT06ARCQ, U19 74LVC2G04LT06ARCQ

Commit message: BOM update
Parts:
- C44, C46, C48, C49, C50: MPN (none) -> FCC0603B104K500CT; now in the parts list
- C45, C47: MPN (none) -> CL10A106MA8NRNC; now in the parts list
- C51: MPN (none) -> CL10B105KA8NNNC; now in the parts list
- D16, D17: MPN (none) -> GL0805UR01
- FB1, FB2: value CBG160808U601T -> 600ohm; MPN (none) -> CBG160808U601T
- J10, J11: MPN (none) -> HL-SMA-KHDC5T
- J12: LCSC# (none) -> C5917305; MPN (none) -> F32258MUBCE2O
- J13: MPN (none) -> MLD-TF PUSH-H18
- J8, J9: MPN (none) -> -
- R55, R56, R57, R58, R59, R60: MPN (none) -> FRC0603F1002TS; now in the parts list
- R61, R62: MPN (none) -> HRC0603F2200ENTN; now in the parts list
- R63, R64: MPN (none) -> RTT035101FTP; now in the parts list
- U16, U17: MPN (none) -> E220-400M22S
- U18, U19: MPN (none) -> 74LVC2G04LT06ARCQ
