File: Board/NNCpro.kicad_sch (KiCad schematic)
At the start: 55 parts, among them U1 W25Q128JVE, U3 boot, U5 RST, U6 STM32H562RIVx, Y1 Crystal_GND24

Commit message: BOM update
Parts:
- C1, C10, C12, C5, C7, C8, C9: MPN (none) -> FCC0603B104K500CT; now in the parts list
- C11, C2: MPN (none) -> CL10B105KA8NNNC; now in the parts list
- C3, C4: MPN (none) -> CL10A225KO8NNNC; now in the parts list
- C6: MPN (none) -> CL10A475KO8NNNC; now in the parts list
- J27, J28, J29, J30, J31, J32, J33, J34, J35, J36, J37, J38, J39, J40, J41, J42, J43, J44, J45, J46, U2, U3, U4, U5: MPN (none) -> -; now left out of the parts list
- L1: MPN (none) -> LQG15HS27NJ02D
- R1, R10, R11, R2, R3, R4, R7, R8, R9: MPN (none) -> FRC0603F1002TS; now in the parts list
- R5, R6: MPN (none) -> HRC0603J472 ENTN; now in the parts list
- TP1, TP2, TP3, TP4: MPN (none) -> -
- U1: MPN (none) -> W25Q128JVE
- U6: MPN (none) -> STM32H562RIV6
- Y1: MPN (none) -> F32258MUBCE2O
