File: Board/Others.kicad_sch (KiCad schematic)
At the start: 54 parts, among them J14 Conn_01x03_Pin, J15 Conn_01x03_Pin, J16 Conn_01x03_Pin, J17 Conn_01x03_Pin, J18 Conn_01x03_Pin, J19 Conn_Coaxial, J20 Conn_01x03_Pin, J21 Conn_01x03_Pin, J22 Conn_01x03_Pin, Q7 DO2300B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

Commit message: BOM update
Parts:
- BZ1: LCSC# (none) -> C781886; MPN (none) -> YX-SMD8530P
- C52, C53, C56: MPN (none) -> FCC0603B104K500CT; now in the parts list
- C54: MPN (none) -> 0603X7R103K250NT; now in the parts list
- C55: MPN (none) -> CL10A106MA8NRNC; now in the parts list
- D18, D19, D20: MPN (none) -> XL-0807RGBC-2812B-S
- D21, D22, D23, D24: MPN (none) -> GL0805UR01
- FB3: value CBG160808U601T -> 600ohm; MPN (none) -> CBG160808U601T
- H1, H2, H3, H4, J14, J15, J16, J17, J18, J20, J21, J22, JP1, JP2, JP3, JP4, JP5, JP6, JP7, JP8: MPN (none) -> -
- J19: MPN (none) -> 5001-RF00001-03R1-00
- L4: value LQG15HS27NJ02D -> 27nH; MPN (none) -> LQG15HS27NJ02D
- Q7: MPN (none) -> DO2300B
- Q8: MPN (none) -> SI1016CX-T1-GE3
- R65, R66, R67, R73, R74: MPN (none) -> HRC0603F2200ENTN; now in the parts list
- R68, R76: MPN (none) -> FRC0603F1002TS; now in the parts list
- R69: MPN (none) -> GR0603J560RT5G00; now in the parts list
- R70, R72: MPN (none) -> CL0603JN100KP; now in the parts list
- R71: MPN (none) -> 1RC0603J0100; now in the parts list
- R75: MPN (none) -> FRC0603F1001TS; now in the parts list
- U20: MPN (none) -> PCA9685BS
- U21: MPN (none) -> LT6000CDCB#TRMPBF
- U22: MPN (none) -> NC7WZ07P6X
- U23: MPN (none) -> MAX-M10M-20B
