File: Board/Power.kicad_sch (KiCad schematic)
At the start: 49 parts, among them IC2 TPS56C230RJER, J1 Screw_Terminal_01x02, U12 TPS564242DRLR, U15 INA3221

Commit message: BOM update
Parts:
- C25, C26, C27, C31, C33: MPN (none) -> CL10A226MP8NUNE; now in the parts list
- C28, C29, C32, C34, C39, C40, C41, C42, C43: MPN (none) -> FCC0603B104K500CT; now in the parts list
- C30: MPN (none) -> CL10B105KA8NNNC; now in the parts list
- C35, C36, C37, C38: MPN (none) -> CL21A476MRYNNNE; now in the parts list
- IC2: MPN (none) -> TPS56C230RJER
- J1: MPN (none) -> KF301-2P; now in the parts list
- L3: MPN (none) -> 7443934450068
- R12: MPN (none) -> GR0603J330KT5G00; now in the parts list
- R13, R20: MPN (none) -> CL0603JN100KP; now in the parts list
- R14, R16: MPN (none) -> SCR0603J15K; now in the parts list
- R15: MPN (none) -> CL0603FN110KP; now in the parts list
- R17: MPN (none) -> RT0603BRD07135KL; now in the parts list
- R18: MPN (none) -> CL0603JN30KP; now in the parts list
- R19: MPN (none) -> RS-03K4222FT; now in the parts list
- R21, R22, R23: MPN (none) -> YLRY06-1-30F; now in the parts list
- R24, R25, R26, R27, R28, R29: MPN (none) -> 1RC0603J0100; now in the parts list
- R30: MPN (none) -> FRC0603F1002TS; now in the parts list
- U12: MPN (none) -> TPS564242DRLR
- U13, U14: MPN (none) -> -; now left out of the parts list
- U15: MPN (none) -> INA3221AIRGVR
