File: Board/Sensors.kicad_sch (KiCad schematic)
At the start: 18 parts, among them IC1 LSM6DSV80XTR, U10 LSM6DSO32, U11 H3LIS200DLTR, U7 MS5611-01BA, U8 BMP390L, U9 MMC5983MA

Commit message: BOM update
Parts:
- C13, C14, C15, C16, C18, C19, C22, C23, C24: MPN (none) -> FCC0603B104K500CT; now in the parts list
- C17, C21: MPN (none) -> CL10A106MA8NRNC; now in the parts list
- C20: MPN (none) -> CL10B105KA8NNNC; now in the parts list
- IC1: MPN (none) -> LSM6DSV80XTR
- U10: MPN (none) -> LSM6DSO32
- U11: MPN (none) -> H3LIS200DLTR
- U7: MPN (none) -> MS5611-01BA
- U8: MPN (none) -> BMP390L
- U9: MPN (none) -> MMC5983MA
